Commit message: adjusted the param for stonefish

File: mvp2_test_robot_description/urdf/base.urdf (robot description, URDF)
Before this commit: robot mvp2_test_robot, 14 links, 13 joints
Joints:
- joint base_link: origin xyz=0.72 0.0 0.0 rpy=0.0 0.0 0.0 -> xyz=0.0 0.0 0.0 rpy=0.0 0.0 0.0
- joint imu__sf_joint: origin xyz=0.0 0.0 0.0 rpy=0.0 0.0 0.0 -> xyz=-0.2 -0.07 0.0 rpy=3.1415926 0.0 0.0; parent imu -> base_link

Commit message: corrected imu_sf tf

File: mvp2_test_robot_description/urdf/base.urdf (robot description, URDF)
Before this commit: robot mvp2_test_robot, 14 links, 13 joints
Joints:
- joint imu__sf_joint: origin xyz=-0.2 -0.07 0.0 rpy=3.1415926 0.0 0.0 -> xyz=-0.2 -0.07 0.0 rpy=0.0 0.0 0.0
- joint imu_joint: origin xyz=-0.2 -0.07 0.0 rpy=3.1415926 0.0 0.0 -> xyz=-0.2 -0.07 0.0 rpy=0.0 0.0 0.0

Commit message: updated config

File: mvp2_test_robot_description/urdf/base.urdf (robot description, URDF)
Before this commit: robot mvp2_test_robot, 15 links, 14 joints
Links:
- removed link usbl
Joints:
- removed joint usbl_joint

Commit message: updated stuff for controller, tf

File: mvp2_test_robot_description/urdf/base.urdf (robot description, URDF)
Before this commit: robot mvp2_test_robot, 14 links, 13 joints
Links:
- added link mbes_link_sf
Joints:
- added joint mbes_link_joint_sf: type fixed, parent nose_tip_link, child mbes_link_sf, origin xyz=0.0 0.0 0.0 rpy=1.5708 0.349 0.0

Commit message: add FLS tf

File: mvp2_test_robot_description/urdf/base.urdf (robot description, URDF)
Before this commit: robot mvp2_test_robot, 15 links, 14 joints
Links:
- added link fls_link_sf
Joints:
- added joint fls_link_joint_sf: type fixed, parent nose_tip_link, child fls_link_sf, origin xyz=0.0 0.0 0.0 rpy=-1.91986218 0.0 -1.57079633

Commit message: add FLS frame in ROS

File: mvp2_test_robot_description/urdf/base.urdf (robot description, URDF)
Before this commit: robot mvp2_test_robot, 16 links, 15 joints
Links:
- added link fls_link_ros
Joints:
- added joint fls_link_joint_ros: type fixed, parent fls_link_sf, child fls_link_ros, origin xyz=0.0 0.0 0.0 rpy=0.0 -1.5707963 0.0

Commit message: fix the fls ros tf

File: mvp2_test_robot_description/urdf/base.urdf (robot description, URDF)
Before this commit: robot mvp2_test_robot, 17 links, 16 joints
Joints:
- joint fls_link_joint_ros: origin xyz=0.0 0.0 0.0 rpy=0.0 -1.5707963 0.0 -> xyz=0.0 0.0 0.0 rpy=-1.5707963 -1.5707963 0.0

Commit message: added gps odom testing

File: mvp2_test_robot_description/urdf/base.urdf (robot description, URDF)
Before this commit: robot mvp2_test_robot, 15 links, 14 joints
Links:
- added link gps2
Joints:
- added joint gps2_joint: type fixed, parent base_link, child gps2, origin xyz=-0.5 0.0 0.32 rpy=3.1415926 0.0 0.0

Commit message: updated with new mvp_mission

File: mvp2_test_robot_description/urdf/base.urdf (robot description, URDF)
Before this commit: robot mvp2_test_robot, 16 links, 15 joints
Links:
- added link usbl
Joints:
- added joint usbl_joint: type fixed, parent base_link, child usbl, origin xyz=0.2 0.0 0.0 rpy=3.1415926 0.0 0.0
